File: flexcable/flexcable.kicad_pcb (KiCad board)
At the start: 2 copper layers, 5.5 x 10.2 mm, 2 parts

Commit message: Day 1
Parts:
- C1, C2: footprint trill-flex:trill_flex_longv2 -> trill-flex:trill_flex_longv3
Routing:
- net Net-(C1-Pad1): track 0.00 -> 37.6 mm, vias 0 -> 1
Other:
- board size 5.5 x 10.2 mm -> 6.8 x 10.2 mm

Commit message: Day 2
Routing:
- net Net-(C1-Pad9): track 0.00 -> 37.6 mm, vias 0 -> 1
- net Net-(C1-Pad8): track 0.00 -> 37.6 mm, vias 0 -> 1
- net Net-(C1-Pad7): track 0.00 -> 37.6 mm, vias 0 -> 1
- net Net-(C1-Pad6): track 0.00 -> 37.6 mm, vias 0 -> 1
- net Net-(C1-Pad5): track 0.00 -> 37.6 mm, vias 0 -> 1
- net Net-(C1-Pad4): track 0.00 -> 37.6 mm, vias 0 -> 1
- net Net-(C1-Pad3): track 0.00 -> 37.6 mm, vias 0 -> 1
- net Net-(C1-Pad2): track 0.00 -> 37.6 mm, vias 0 -> 1
- net Net-(C1-Pad10): track 0.00 -> 37.6 mm, vias 0 -> 1
- added copper zone on B.Cu, net (none)
- added copper zone on F.Cu, net (none)
Changed lines of the file:
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@@
 	)
 	(paper "A4")
+	(title_block
+		(title "Google Nest Mini Gen 2 Flex Cable")
+		(date "2025-09-10")
+		(rev "v1.0")
+	)
 	(layers
 		(0 "F.Cu" signal)
@@
 		(allow_soldermask_bridges_in_footprints no)
 		(tenting front back)
-		(grid_origin 60.92 60.4775)
+		(grid_origin 66.32 60.4775)
 		(pcbplotparams
 			(layerselection 0x00000000_00000000_55555555_5755f5ff)
@@
 	)
 	(segment
+		(start 61.52 69.4775)
+		(end 61.52 87.4775)
+		(width 0.2)
+		(layer "F.Cu")
+		(net 1)
+	)
+	(via
+		(at 61.52 87.4775)
+		(size 0.6)
+		(drill 0.3)
+		(layers "F.Cu" "B.Cu")
+		(net 1)
+	)
+	(segment
+		(start 61.52 107.1175)
+		(end 61.52 87.4775)
+		(width 0.2)
+		(layer "B.Cu")
+		(net 1)
+	)
+	(segment
 		(start 60.92 69.4775)
 		(end 60.92 88.4775)
@@
 		(net 2)
 	)
+	(segment
+		(start 62.12 69.4775)
+		(end 62.12 86.4775)
+		(width 0.2)
+		(layer "F.Cu")
+		(net 3)
+	)
+	(via
+		(at 62.12 86.4775)
+		(size 0.6)
+		(drill 0.3)
+		(layers "F.Cu" "B.Cu")
+		(net 3)
+	)
+	(segment
+		(start 62.12 107.1175)
+		(end 62.12 86.4775)
+		(width 0.2)
+		(layer "B.Cu")
+		(net 3)
+	)
+	(segment
+		(start 62.72 69.4775)
+		(end 62.72 85.4775)
+		(width 0.2)
+		(layer "F.Cu")
+		(net 4)
+	)
+	(via
+		(at 62.72 85.4775)
+		(size 0.6)
+		(drill 0.3)
+		(layers "F.Cu" "B.Cu")
+		(net 4)
+	)
+	(segment
+		(start 62.72 107.1175)
+		(end 62.72 85.4775)
+		(width 0.2)
+		(layer "B.Cu")
+		(net 4)
+	)
+	(segment
+		(start 63.32 69.4775)
+		(end 63.32 84.4775)
+		(width 0.2)
+		(layer "F.Cu")
+		(net 5)
+	)
+	(via
+		(at 63.32 84.4775)
+		(size 0.6)
+		(drill 0.3)
+		(layers "F.Cu" "B.Cu")
+		(net 5)
+	)
+	(segment
+		(start 63.32 107.1175)
+		(end 63.32 84.4775)
+		(width 0.2)
+		(layer "B.Cu")
+		(net 5)
+	)
+	(segment
+		(start 65.12 69.4775)
+		(end 65.12 81.4775)
+		(width 0.2)
+		(layer "F.Cu")
+		(net 6)
+	)
+	(via
+		(at 65.12 81.4775)
+		(size 0.6)
+		(drill 0.3)
+		(layers "F.Cu" "B.Cu")
+		(net 6)
+	)
+	(segment
+		(start 65.12 107.1175)
+		(end 65.12 81.4775)
+		(width 0.2)
+		(layer "B.Cu")
+		(net 6)
+	)
+	(segment
+		(start 66.32 69.4775)
+		(end 66.32 79.4775)
+		(width 0.2)
+		(layer "F.Cu")
+		(net 7)
+	)
+	(via
+		(at 66.32 79.4775)
+		(size 0.6)
+		(drill 0.3)
+		(layers "F.Cu" "B.Cu")
+		(net 7)
+	)
+	(segment
+		(start 66.32 107.1175)
+		(end 66.32 79.4775)
+		(width 0.2)
+		(layer "B.Cu")
+		(net 7)
+	)
+	(segment
+		(start 65.72 69.4775)
+		(end 65.72 80.4775)
+		(width 0.2)
+		(layer "F.Cu")
+		(net 8)
+	)
+	(via
+		(at 65.72 80.4775)
+		(size 0.6)
+		(drill 0.3)
+		(layers "F.Cu" "B.Cu")
+		(net 8)
+	)
+	(segment
+		(start 65.72 107.1175)
+		(end 65.72 80.4775)
+		(width 0.2)
+		(layer "B.Cu")
+		(net 8)
+	)
+	(segment
+		(start 63.92 69.4775)
+		(end 63.92 83.4775)
+		(width 0.2)
+		(layer "F.Cu")
+		(net 9)
+	)
+	(via
+		(at 63.92 83.4775)
+		(size 0.6)
+		(drill 0.3)
+		(layers "F.Cu" "B.Cu")
+		(net 9)
+	)
+	(segment
+		(start 63.92 107.1175)
+		(end 63.92 83.4775)
+		(width 0.2)
+		(layer "B.Cu")
+		(net 9)
+	)
+	(segment
+		(start 64.52 69.4775)
+		(end 64.52 82.4775)
+		(width 0.2)
+		(layer "F.Cu")
+		(net 10)
+	)
+	(via
+		(at 64.52 82.4775)
+		(size 0.6)
+		(drill 0.3)
+		(layers "F.Cu" "B.Cu")
+		(net 10)
+	)
+	(segment
+		(start 64.52 107.1175)
+		(end 64.52 82.4775)
+		(width 0.2)
+		(layer "B.Cu")
+		(net 10)
+	)
+	(zone
+		(net 0)
+		(net_name "")
+		(layers "F.Cu" "B.Cu")
+		(hatch edge 0.5)
+		(connect_pads
+			(clearance 0.5)
+		)
+		(min_thickness 0.25)
+		(filled_areas_thickness no)
+		(fill yes
+			(thermal_gap 0.5)
+			(thermal_bridge_width 0.5)
+			(island_removal_mode 1)
+			(island_area_min 10)
+		)
+		(polygon
+			(pts
+				(xy 60.195 60.2975) (xy 67.06 60.2975) (xy 67.06 116.294175) (xy 60.195 116.294175)
+			)
+		)
+	)
 	(embedded_fonts no)
