File: flexcable/flexcable.kicad_sch (KiCad schematic)
At the start: 2 parts

Commit message: Part 1.1
Connections:
- new net: C1.10, C2.10
- new net: C1.6, C2.6
- new net: C1.7, C2.7
- new net: C1.8, C2.8
- new net: C1.9, C2.9
Changed lines of the file:
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@@
 			)
 		)
-		(pin "18"
+		(pin "9"
 		)
-		(pin "20"
+		(pin "6"
 		)
 		(pin "4"
 		)
-		(pin "17"
+		(pin "7"
 		)
 		(pin "2"
 		)
-		(pin "21"
+		(pin "10"
 		)
 		(pin "5"
@@
 		(pin "3"
 		)
-		(pin "19"
+		(pin "8"
 		)
 		(instances
@@
 	)
 	(symbol
+		(lib_name "trill-flex-conector_1")
 		(lib_id "trill-flex:trill-flex-conector")
 		(at 49.53 36.83 0)
@@
 			)
 		)
-		(pin "18"
+		(pin "7"
 		)
-		(pin "20"
+		(pin "10"
 		)
 		(pin "4"
 		)
-		(pin "17"
+		(pin "8"
 		)
 		(pin "2"
 		)
-		(pin "21"
+		(pin "6"
 		)
 		(pin "5"
@@
 		(pin "3"
 		)
-		(pin "19"
+		(pin "9"
 		)
 		(instances

Commit message: Day 1
Parts:
- C1, C2: footprint trill-flex:trill_flex_longv2 -> trill-flex:trill_flex_longv3
Changed lines of the file:
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@@
 			)
 		)
-		(property "Footprint" "trill-flex:trill_flex_longv2"
+		(property "Footprint" "trill-flex:trill_flex_longv3"
 			(at 49.53 59.69 0)
 			(effects
@@
 			)
 		)
-		(property "Footprint" "trill-flex:trill_flex_longv2"
+		(property "Footprint" "trill-flex:trill_flex_longv3"
 			(at 49.53 36.83 0)
 			(effects

Commit message: Day 2
Other:
- title: (none) -> Google Nest Mini Gen 2 Flex Cable
Changed lines of the file:
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@@
 	(generator_version "9.0")
 	(paper "A4")
+	(title_block
+		(title "Google Nest Mini Gen 2 Flex Cable")
+		(date "2025-09-10")
+		(rev "v1.1")
+	)
 	(wire
 		(pts
